File: Labor Netzteil.sch (KiCad schematic (older format))
At the start: 14 parts

Commit message: Neuigkeiten
Parts:
- removed J?: Fan, symbol Connector_Generic:Conn_01x02
- removed J?: ESP Board, symbol Connector_Generic:Conn_01x02
- added D? (x2): D, symbol Device:D
- added J1: Out02, symbol Connector_Generic:Conn_01x01
- added J10: Sec 2 d, symbol Connector_Generic:Conn_01x01
- added J11, J12: Conn_01x01, symbol Connector_Generic:Conn_01x01
- added J16: Fan, symbol Connector_Generic:Conn_01x04
- added J2: Out01, symbol Connector_Generic:Conn_01x01
- added J3: Sec 1 d, symbol Connector_Generic:Conn_01x01
- added J4: Sec 1 c, symbol Connector_Generic:Conn_01x01
- added J5: Sec 1 b, symbol Connector_Generic:Conn_01x01
- added J6: Sec 1 a, symbol Connector_Generic:Conn_01x01
- added J7: Sec 2 a, symbol Connector_Generic:Conn_01x01
- added J8: Sec 2 b, symbol Connector_Generic:Conn_01x01
- added J9: Sec 2 c, symbol Connector_Generic:Conn_01x01
- added J?: OLED, symbol Connector_Generic:Conn_01x04
- added K1, K2: G5LE-1, Relay_THT:Relay_SPDT_Omron-G5LE-1, symbol Relay:G5LE-1
- added U?: ESP-DevKitC, symbol ESP32-DevKitC:ESP-DevKitC
- C2, C3: renamed from C?; value C -> 0,33uF
- C4, C5: renamed from C?; value C -> 0,1uF
- gave numbers to parts that had none: 8
Connections:
- net GND: now reaches C1.1, C2.1, C3.1, D1.1 (K), D2.1 (K), U1.1 (VI), U2.1 (VI)
- net GND: now also D?.2 (A), D?.2 (A), J16.4 (Pin_4), J?.4 (Pin_4), K1.5, K2.5, U?.14 (GND), U?.32 (GND)
- net 12V: now reaches U1.3 (VO)
- net 12V: now also C5.1, J16.1 (Pin_1); no longer C4.1
- net 5V: now reaches U2.3 (VO)
- net 5V: now also C4.1, U?.19 (5V); no longer C5.1
- new net: J1.1 (Pin_1), K1.1
- new net: D?.1 (K), K1.2
- new net: J3.1 (Pin_1), K1.3
- new net: J4.1 (Pin_1), J5.1 (Pin_1), K1.4
- new net: J12.1 (Pin_1), K2.1
- new net: D?.1 (K), K2.2
- new net: J10.1 (Pin_1), K2.3
- new net: J8.1 (Pin_1), J9.1 (Pin_1), K2.4
- new net: J2.1 (Pin_1), J6.1 (Pin_1)
- new net: J11.1 (Pin_1), J7.1 (Pin_1)
- new net 3V3: J?.1 (Pin_1), U?.1 (3V3)
- new net SCL: J?.3 (Pin_3), U?.36 (22)
- new net SDA: J?.2 (Pin_2), U?.33 (21)
Other:
- moved on the sheet: U1, U2
