File: kicad/Labor Netzteil.sch (KiCad schematic (older format))
At the start: 31 parts, among them J1 Out02, J10 Sec 2 d, J11 Conn_01x01, J12 Conn_01x01, J13 Conn_01x02, J16 Fan, J2 Out01, J3 Sec 1 d, J4 Sec 1 c, J5 Sec 1 b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

Commit message: Relais Modul und Level Shifter hinzugefügt
Parts:
- removed D? (x2): D, symbol Device:D
- removed K1, K2: G5LE-1, Relay_THT:Relay_SPDT_Omron-G5LE-1, symbol Relay:G5LE-1
- added U1: 2-Relais-Modul, symbol Relais~Modul:2-Relais-Modul
- added U5: 74HC245, symbol 74xx:74HC245
- gave numbers to parts that had none: 2
- renumbered J16 to J15, U1 to U3
Connections:
- net labels added: A0, A1, B0, B1
- wire segments 98 -> 112
Other:
- moved on the sheet: J10, J11, J12, J7, J8, J9

Commit message: Leiterplatte im Prinzip fertig
Parts:
- removed J13: Conn_01x02, symbol Connector_Generic:Conn_01x02
- added J15: Out_1, Connector_Pin:Pin_D1.0mm_L10.0mm, symbol Connector_Generic:Conn_01x01
- added J16: NeoPixel, Connector_JST:JST_XH_B3B-XH-A_1x03_P2.50mm_Vertical, symbol Connector_Generic:Conn_01x03
- added J17: Out_2, Connector_Pin:Pin_D1.0mm_L10.0mm, symbol Connector_Generic:Conn_01x01
- added R1, R4: 10k, Resistor_THT:R_Axial_DIN0207_L6.3mm_D2.5mm_P10.16mm_Horizontal, symbol Device:R
- added R2, R3, R5: 1k, Resistor_THT:R_Axial_DIN0207_L6.3mm_D2.5mm_P10.16mm_Horizontal, symbol Device:R
- added U6: DS18B20, Package_TO_SOT_THT:TO-92_Inline, symbol Sensor_Temperature:DS18B20
- C1: footprint (none) -> Capacitor_THT:CP_Radial_D14.0mm_P5.00mm
- C2, C3, C4, C5: footprint (none) -> Capacitor_THT:C_Disc_D4.7mm_W2.5mm_P5.00mm
- D1, D2, D3, D4: footprint (none) -> Diode_THT:D_5W_P12.70mm_Horizontal
- J1: value Out02 -> Out_1_01; footprint (none) -> Connector_Pin:Pin_D1.3mm_L11.0mm_LooseFit
- J10, J3, J4, J5, J6, J7, J8, J9: footprint (none) -> Connector_Pin:Pin_D1.3mm_L11.0mm_LooseFit
- J11: value Conn_01x01 -> Out_2_02; footprint (none) -> Connector_Pin:Pin_D1.3mm_L11.0mm_LooseFit
- J12: value Conn_01x01 -> Out_2_01; footprint (none) -> Connector_Pin:Pin_D1.3mm_L11.0mm_LooseFit
- J13: renamed from J14; footprint (none) -> Connector_JST:JST_XH_B4B-XH-A_1x04_P2.50mm_Vertical
- J14: renamed from J15; footprint (none) -> Connector_JST:JST_XH_B4B-XH-A_1x04_P2.50mm_Vertical
- J2: value Out01 -> Out_1_02; footprint (none) -> Connector_Pin:Pin_D1.3mm_L11.0mm_LooseFit
- U1: footprint (none) -> Relais Modul:2-way-relais-module
- U4: footprint (none) -> ESP32-DevKitC:ESP32-DevKitC
- U5: footprint (none) -> Package_DIP:DIP-20_W7.62mm_LongPads
Connections:
- net labels added: DS18B20, NeoPixel, PWM, TACHO, V_MON_1, V_MON_2
- wire segments 112 -> 157
- no-connect marks 0 -> 31

Commit message: Leiterplatte Verbesserungen
Parts:
- added C6: 1000uF, Capacitor_THT:CP_Radial_D14.0mm_P5.00mm, symbol Device:CP
- added R6: 470, Resistor_THT:R_Axial_DIN0207_L6.3mm_D2.5mm_P10.16mm_Horizontal, symbol Device:R
- D1, D2, D3, D4: value D -> 1N5400
Connections:
- wire segments 157 -> 168
Other:
- moved on the sheet: D1, D2, D3, D4, J16
Changed lines of the file:
@@
 L Device:D D1
 U 1 1 5E751960
-P 2600 4950
-F 0 "D1" H 2500 4900 50  0000 C CNN
-F 1 "D" H 2700 4900 50  0000 C CNN
-F 2 "Diode_THT:D_5W_P12.70mm_Horizontal" H 2600 4950 50  0001 C CNN
-F 3 "~" H 2600 4950 50  0001 C CNN
-	1    2600 4950
-	-1   0    0    1
-$EndComp
-$Comp
-L Device:D D2
-U 1 1 5E752767
-P 2600 5150
-F 0 "D2" H 2500 5100 50  0000 C CNN
-F 1 "D" H 2700 5100 50  0000 C CNN
-F 2 "Diode_THT:D_5W_P12.70mm_Horizontal" H 2600 5150 50  0001 C CNN
-F 3 "~" H 2600 5150 50  0001 C CNN
-	1    2600 5150
+P 2450 4950
+F 0 "D1" H 2550 5000 50  0000 C CNN
+F 1 "1N5400" H 2650 4900 50  0000 C CNN
+F 2 "Diode_THT:D_5W_P12.70mm_Horizontal" H 2450 4950 50  0001 C CNN
+F 3 "~" H 2450 4950 50  0001 C CNN
+	1    2450 4950
 	-1   0    0    1
 $EndComp
@@
 L Device:D D3
 U 1 1 5E753466
-P 2600 5350
-F 0 "D3" H 2700 5400 50  0000 C CNN
-F 1 "D" H 2500 5400 50  0000 C CNN
-F 2 "Diode_THT:D_5W_P12.70mm_Horizontal" H 2600 5350 50  0001 C CNN
-F 3 "~" H 2600 5350 50  0001 C CNN
-	1    2600 5350
+P 2450 5350
+F 0 "D3" H 2350 5300 50  0000 C CNN
+F 1 "1N5400" H 2250 5400 50  0000 C CNN
+F 2 "Diode_THT:D_5W_P12.70mm_Horizontal" H 2450 5350 50  0001 C CNN
+F 3 "~" H 2450 5350 50  0001 C CNN
+	1    2450 5350
 	1    0    0    -1
 $EndComp
@@
 L Device:D D4
 U 1 1 5E75388D
-P 2600 5550
-F 0 "D4" H 2700 5600 50  0000 C CNN
-F 1 "D" H 2500 5600 50  0000 C CNN
-F 2 "Diode_THT:D_5W_P12.70mm_Horizontal" H 2600 5550 50  0001 C CNN
-F 3 "~" H 2600 5550 50  0001 C CNN
-	1    2600 5550
+P 2450 5550
+F 0 "D4" H 2350 5500 50  0000 C CNN
+F 1 "1N5400" H 2250 5600 50  0000 C CNN
+F 2 "Diode_THT:D_5W_P12.70mm_Horizontal" H 2450 5550 50  0001 C CNN
+F 3 "~" H 2450 5550 50  0001 C CNN
+	1    2450 5550
 	1    0    0    -1
 $EndComp
 Connection ~ 3500 4950
 Wire Wire Line
-	2450 5050 2450 5150
-Wire Wire Line
 	3500 4950 3500 6350
 Wire Wire Line
 	1800 4950 1800 5350
 Wire Wire Line
-	1800 5350 2450 5350
-Wire Wire Line
-	1800 4950 2450 4950
-Wire Wire Line
-	2000 5050 2000 5550
-Wire Wire Line
-	2000 5550 2450 5550
-Wire Wire Line
-	2000 5050 2450 5050
-Wire Wire Line
-	2750 5350 2750 5550
-Wire Wire Line
-	2750 4950 2750 5150
-Connection ~ 2750 4950
-Wire Wire Line
-	2750 5550 2750 5950
-Connection ~ 2750 5550
+	1800 5350 2300 5350
+Wire Wire Line
+	1800 4950 2300 4950
+Wire Wire Line
+	2000 5150 2000 5550
+Wire Wire Line
+	2000 5550 2300 5550
 Wire Wire Line
 	2750 5950 3050 5950
@@
 	2750 7350 4250 7350
 Wire Wire Line
-	2750 4950 3050 4950
+	2600 4950 2750 4950
 $Comp
 L Device:CP C1
@@
 L Connector_Generic:Conn_01x03 J16
 U 1 1 5E76A778
-P 8850 1550
-F 0 "J16" V 8850 1850 50  0000 R CNN
-F 1 "NeoPixel" V 8950 1700 50  0000 R CNN
-F 2 "Connector_JST:JST_XH_B3B-XH-A_1x03_P2.50mm_Vertical" H 8850 1550 50  0001 C CNN
-F 3 "~" H 8850 1550 50  0001 C CNN
-	1    8850 1550
-	0    -1   -1   0
+P 10350 1900
+F 0 "J16" V 10350 2200 50  0000 R CNN
+F 1 "NeoPixel" V 10450 2050 50  0000 R CNN
+F 2 "Connector_JST:JST_XH_B3B-XH-A_1x03_P2.50mm_Vertical" H 10350 1900 50  0001 C CNN
+F 3 "~" H 10350 1900 50  0001 C CNN
+	1    10350 1900
+	1    0    0    -1
 $EndComp
 $Comp
 L power:GND #PWR010
 U 1 1 5E76BF25
-P 8950 2250
-F 0 "#PWR010" H 8950 2000 50  0001 C CNN
-F 1 "GND" H 8955 2077 50  0000 C CNN
-F 2 "" H 8950 2250 50  0001 C CNN
-F 3 "" H 8950 2250 50  0001 C CNN
-	1    8950 2250
-	1    0    0    -1
-$EndComp
-Wire Wire Line
-	8950 2250 8950 1750
-Text GLabel 8750 2300 3    50   Input ~ 0
+P 9100 2400
+F 0 "#PWR010" H 9100 2150 50  0001 C CNN
+F 1 "GND" H 9105 2227 50  0000 C CNN
+F 2 "" H 9100 2400 50  0001 C CNN
+F 3 "" H 9100 2400 50  0001 C CNN
+	1    9100 2400
+	1    0    0    -1
+$EndComp
+Text GLabel 9900 1500 1    50   Input ~ 0
 5V
-Wire Wire Line
-	8750 2300 8750 1750
-Text GLabel 8850 1900 3    50   Input ~ 0
+Text GLabel 9400 1500 1    50   Input ~ 0
 NeoPixel
-Wire Wire Line
-	8850 1750 8850 1900
 Wire Wire Line
 	6550 3900 6450 3900
@@
 NoConn ~ 4550 1650
 Wire Wire Line
-	2000 5050 2000 4150
-Connection ~ 2000 5050
+	2000 5150 2000 4150
+Connection ~ 2000 5150
 Connection ~ 2000 4150
 Wire Wire Line
@@
 Wire Wire Line
 	4450 2550 4550 2550
+Wire Wire Line
+	2000 5150 2300 5150
+$Comp
+L Device:D D2
+U 1 1 5E752767
+P 2450 5150
+F 0 "D2" H 2550 5200 50  0000 C CNN
+F 1 "1N5400" H 2650 5100 50  0000 C CNN
+F 2 "Diode_THT:D_5W_P12.70mm_Horizontal" H 2450 5150 50  0001 C CNN
+F 3 "~" H 2450 5150 50  0001 C CNN
+	1    2450 5150
+	-1   0    0    1
+$EndComp
+Wire Wire Line
+	2750 5950 2750 5550
+Wire Wire Line
+	2750 5350 2600 5350
+Wire Wire Line
+	2600 5550 2750 5550
+Connection ~ 2750 5550
+Wire Wire Line
+	2750 5550 2750 5350
+Wire Wire Line
+	2600 5150 2750 5150
+Wire Wire Line
+	2750 5150 2750 4950
+Connection ~ 2750 4950
+Wire Wire Line
+	2750 4950 3050 4950
+$Comp
+L Device:CP C6
+U 1 1 5E7A5B0A
+P 9100 1950
+F 0 "C6" H 9218 1996 50  0000 L CNN
+F 1 "1000uF" H 9218 1905 50  0000 L CNN
+F 2 "Capacitor_THT:CP_Radial_D14.0mm_P5.00mm" H 9138 1800 50  0001 C CNN
+F 3 "~" H 9100 1950 50  0001 C CNN
+	1    9100 1950
+	1    0    0    -1
+$EndComp
+Wire Wire Line
+	9100 2100 9100 2200
+Wire Wire Line
+	9100 2200 9900 2200
+Wire Wire Line
+	9900 2200 9900 2000
+Wire Wire Line
+	9900 2000 10150 2000
+Wire Wire Line
+	9100 2200 9100 2400
+Connection ~ 9100 2200
+Wire Wire Line
+	10150 1800 9900 1800
+Wire Wire Line
+	9900 1800 9900 1500
+$Comp
+L Device:R R6
+U 1 1 5E7DD871
+P 9750 1900
+F 0 "R6" V 9543 1900 50  0000 C CNN
+F 1 "470" V 9634 1900 50  0000 C CNN
+F 2 "Resistor_THT:R_Axial_DIN0207_L6.3mm_D2.5mm_P10.16mm_Horizontal" V 9680 1900 50  0001 C CNN
+F 3 "~" H 9750 1900 50  0001 C CNN
+	1    9750 1900
+	0    1    1    0
+$EndComp
+Wire Wire Line
+	9900 1900 10150 1900
+Wire Wire Line
+	9600 1900 9400 1900
+Wire Wire Line
+	9400 1900 9400 1500
+Text GLabel 9100 1500 1    50   Input ~ 0
+5V
+Wire Wire Line
+	9100 1800 9100 1500
 $EndSCHEMATC

Commit message: aktuellste Lieferungen und Anpassungen
Parts:
- removed U3: LM7812_TO220, Package_TO_SOT_THT:TO-220-3_Vertical, symbol Regulator_Linear:LM7812_TO220
- added C7: 470uF/25V, Capacitor_THT:CP_Radial_D8.0mm_P3.80mm, symbol Device:CP
- added U3: L7812, Package_TO_SOT_THT:TO-220-3_Vertical, symbol Regulator_Linear:L7812
Connections:
- wire segments 168 -> 175
- no-connect marks 31 -> 29
Changed lines of the file:
@@
 $EndDescr
-$Comp
-L Regulator_Linear:LM7812_TO220 U3
-U 1 1 5E7394C5
-P 4650 6350
-F 0 "U3" H 4650 6592 50  0000 C CNN
-F 1 "LM7812_TO220" H 4650 6501 50  0000 C CNN
-F 2 "Package_TO_SOT_THT:TO-220-3_Vertical" H 4650 6575 50  0001 C CIN
-F 3 "${KICAD_DATASHEETS}cd00000444-1795274.pdf" H 4650 6300 50  0001 C CNN
-	1    4650 6350
-	1    0    0    -1
-$EndComp
 $Comp
 L Device:C C2
@@
 5V
 Wire Wire Line
-	4350 3350 4550 3350
+	4350 3350 4450 3350
 Text GLabel 5750 6350 2    50   Input ~ 0
 12V
@@
 Wire Wire Line
 	5150 4950 5750 4950
-NoConn ~ 3750 2800
-NoConn ~ 3750 2900
 Text GLabel 8150 2000 3    50   Input ~ 0
 TACHO
@@
 Wire Wire Line
 	9100 1800 9100 1500
+$Comp
+L Regulator_Linear:L7812 U3
+U 1 1 5E7954AD
+P 4650 6350
+F 0 "U3" H 4650 6592 50  0000 C CNN
+F 1 "L7812" H 4650 6501 50  0000 C CNN
+F 2 "Package_TO_SOT_THT:TO-220-3_Vertical" H 4675 6200 50  0001 L CIN
+F 3 "http://www.st.com/content/ccc/resource/technical/document/datasheet/41/4f/b3/b0/12/d4/47/88/CD00000444.pdf/files/CD00000444.pdf/jcr:content/translations/en.CD00000444.pdf" H 4650 6300 50  0001 C CNN
+	1    4650 6350
+	1    0    0    -1
+$EndComp
+$Comp
+L Device:CP C7
+U 1 1 5E7A0326
+P 5150 3800
+F 0 "C7" H 5268 3846 50  0000 L CNN
+F 1 "470uF/25V" H 5268 3755 50  0000 L CNN
+F 2 "Capacitor_THT:CP_Radial_D8.0mm_P3.80mm" H 5188 3650 50  0001 C CNN
+F 3 "~" H 5150 3800 50  0001 C CNN
+	1    5150 3800
+	1    0    0    -1
+$EndComp
+Wire Wire Line
+	5150 3650 4450 3650
+Wire Wire Line
+	4450 3650 4450 3350
+Connection ~ 4450 3350
+Wire Wire Line
+	4450 3350 4550 3350
+$Comp
+L power:GND #PWR0101
+U 1 1 5E7A9F82
+P 5150 4150
+F 0 "#PWR0101" H 5150 3900 50  0001 C CNN
+F 1 "GND" H 5155 3977 50  0000 C CNN
+F 2 "" H 5150 4150 50  0001 C CNN
+F 3 "" H 5150 4150 50  0001 C CNN
+	1    5150 4150
+	1    0    0    -1
+$EndComp
+Wire Wire Line
+	5150 4150 5150 3950
+Wire Wire Line
+	3750 2800 3800 2800
+Wire Wire Line
+	3800 2800 3800 2900
+Wire Wire Line
+	3800 2900 3750 2900
 $EndSCHEMATC
