File: kicad/Labor Netzteil.kicad_sch (KiCad schematic)
At the start: 40 parts, among them J1 Out_1_01, J10 Sec 2 d, J11 Out_2_02, J12 Out_2_01, J13 OLED, J14 Fan, J15 Out_1, J16 NeoPixel, J17 Out_2, J2 Out_1_02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

Commit message: Added PS module datasheet
Changed lines of the file:
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@@
     (stroke (width 0) (type default))
   )
-  (wire (pts (xy 109.22 54.61) (xy 115.57 54.61))
+  (wire (pts (xy 109.855 54.61) (xy 115.57 54.61))
     (stroke (width 0) (type default))
   )
@@
     (stroke (width 0) (type default))
   )
-  (wire (pts (xy 95.25 60.96) (xy 99.06 60.96))
-    (stroke (width 0) (type default))
-  )
-  (wire (pts (xy 109.22 49.53) (xy 115.57 49.53))
-    (stroke (width 0) (type default))
-  )
-  (wire (pts (xy 115.57 62.23) (xy 113.03 62.23))
-    (stroke (width 0) (type default))
-  )
-  (wire (pts (xy 95.25 58.42) (xy 99.06 58.42))
+  (wire (pts (xy 95.25 60.96) (xy 98.425 60.96))
+    (stroke (width 0) (type default))
+  )
+  (wire (pts (xy 109.855 49.53) (xy 115.57 49.53))
+    (stroke (width 0) (type default))
+  )
+  (wire (pts (xy 115.57 62.23) (xy 113.665 62.23))
+    (stroke (width 0) (type default))
+  )
+  (wire (pts (xy 95.25 58.42) (xy 98.425 58.42))
     (stroke (width 0) (type default))
   )
@@
     (stroke (width 0) (type default))
   )
-  (wire (pts (xy 113.03 64.77) (xy 115.57 64.77))
+  (wire (pts (xy 113.665 64.77) (xy 115.57 64.77))
     (stroke (width 0) (type default))
   )
@@
     (stroke (width 0) (type default))
   )
-  (wire (pts (xy 109.22 52.07) (xy 115.57 52.07))
+  (wire (pts (xy 109.855 52.07) (xy 115.57 52.07))
     (stroke (width 0) (type default))
   )
@@
     )
   )
-  (global_label "A1" (shape input) (at 109.22 52.07 180)
-    (effects (font (size 1.27 1.27)) (justify right))
-    (property "Intersheetrefs" "${INTERSHEET_REFS}" (at 109.22 52.07 0)
+  (global_label "A1" (shape input) (at 109.855 52.07 180)
+    (effects (font (size 1.27 1.27)) (justify right))
+    (property "Intersheetrefs" "${INTERSHEET_REFS}" (at 109.855 52.07 0)
       (effects (font (size 1.27 1.27)) hide)
     )
@@
     )
   )
-  (global_label "B0" (shape input) (at 99.06 60.96 0)
-    (effects (font (size 1.27 1.27)) (justify left))
-    (property "Intersheetrefs" "${INTERSHEET_REFS}" (at 99.06 60.96 0)
+  (global_label "B0" (shape input) (at 98.425 60.96 0)
+    (effects (font (size 1.27 1.27)) (justify left))
+    (property "Intersheetrefs" "${INTERSHEET_REFS}" (at 98.425 60.96 0)
       (effects (font (size 1.27 1.27)) hide)
     )
@@
     )
   )
-  (global_label "A0" (shape input) (at 109.22 49.53 180)
-    (effects (font (size 1.27 1.27)) (justify right))
-    (property "Intersheetrefs" "${INTERSHEET_REFS}" (at 109.22 49.53 0)
+  (global_label "A0" (shape input) (at 109.855 49.53 180)
+    (effects (font (size 1.27 1.27)) (justify right))
+    (property "Intersheetrefs" "${INTERSHEET_REFS}" (at 109.855 49.53 0)
       (effects (font (size 1.27 1.27)) hide)
     )
@@
     )
   )
-  (global_label "V_MON_2" (shape input) (at 113.03 64.77 180)
-    (effects (font (size 1.27 1.27)) (justify right))
-    (property "Intersheetrefs" "${INTERSHEET_REFS}" (at 113.03 64.77 0)
+  (global_label "V_MON_2" (shape input) (at 113.665 64.77 180)
+    (effects (font (size 1.27 1.27)) (justify right))
+    (property "Intersheetrefs" "${INTERSHEET_REFS}" (at 113.665 64.77 0)
       (effects (font (size 1.27 1.27)) hide)
     )
@@
     )
   )
-  (global_label "B1" (shape input) (at 99.06 58.42 0)
-    (effects (font (size 1.27 1.27)) (justify left))
-    (property "Intersheetrefs" "${INTERSHEET_REFS}" (at 99.06 58.42 0)
+  (global_label "B1" (shape input) (at 98.425 58.42 0)
+    (effects (font (size 1.27 1.27)) (justify left))
+    (property "Intersheetrefs" "${INTERSHEET_REFS}" (at 98.425 58.42 0)
       (effects (font (size 1.27 1.27)) hide)
     )
@@
     )
   )
-  (global_label "NeoPixel" (shape input) (at 109.22 54.61 180)
-    (effects (font (size 1.27 1.27)) (justify right))
-    (property "Intersheetrefs" "${INTERSHEET_REFS}" (at 109.22 54.61 0)
+  (global_label "NeoPixel" (shape input) (at 109.855 54.61 180)
+    (effects (font (size 1.27 1.27)) (justify right))
+    (property "Intersheetrefs" "${INTERSHEET_REFS}" (at 109.855 54.61 0)
       (effects (font (size 1.27 1.27)) hide)
     )
@@
     )
   )
-  (global_label "V_MON_1" (shape input) (at 113.03 62.23 180)
-    (effects (font (size 1.27 1.27)) (justify right))
-    (property "Intersheetrefs" "${INTERSHEET_REFS}" (at 113.03 62.23 0)
-      (effects (font (size 1.27 1.27)) hide)
-    )
+  (global_label "V_MON_1" (shape input) (at 113.665 62.23 180)
+    (effects (font (size 1.27 1.27)) (justify right))
+    (property "Intersheetrefs" "${INTERSHEET_REFS}" (at 113.665 62.23 0)
+      (effects (font (size 1.27 1.27)) hide)
+    )
